File: v1.2/Croduino Nova v1.2.sch (EAGLE design)
At the start: 40 parts, among them IC1 CP210X_USB_UART, Q1 MMBT2222A, Q2 MMBT2222A, U2 SE5218-3.3V, X1 ESP8266-12

Commit message: added v1.2 version
Parts:
- removed D2: MBR0520LT, diode:MBR0520LT
- added D1: BAT20J, SparkFun-DiscreteSemi:DIODE-SCHOTTKY-BAT20J
- added Q3: PMOS, SparkFun-DiscreteSemi:MOSFET_PCH-IRLML2244
- added R13: 100k, SparkFun-Resistors:100KOHM-0603-1/10W-1%
Connections:
- new net V_USB: D1.A, F1.2, Q3.G, R13.2
- net BAT: now also Q3.D; no longer D2.A
- net GND: now also R13.1, U$7.TEMP
- net VCC: now also D1.C, Q3.S; no longer D2.C, F1.2
Other:
- note added: "3.3V Voltage Regulator"
- note added: "Automatic source selection"
- note added: "Battery Charger"
- moved on the sheet: C1, C7, JP8, U2
